Commit message: Updated compatible version to 2.49.0

File: realsense2_description/urdf/_d415.urdf.xacro (robot description, xacro)
@@ -1,19 +1,6 @@
 <?xml version="1.0"?>
 <!--
-# Copyright 2023 Intel Corporation. All Rights Reserved.
-#
-# Licensed under the Apache License, Version 2.0 (the "License");
-# you may not use this file except in compliance with the License.
-# You may obtain a copy of the License at
-#
-#     http://www.apache.org/licenses/LICENSE-2.0
-#
-# Unless required by applicable law or agreed to in writing, software
-# distributed under the License is distributed on an "AS IS" BASIS,
-# WITHOUT WARRANTIES OR CONDITIONS OF ANY KIND, either express or implied.
-# See the License for the specific language governing permissions and
-# limitations under the License.
--->
-<!--
+License: Apache 2.0. See LICENSE file in root directory.
+Copyright(c) 2017 Intel Corporation. All Rights Reserved
 This is the URDF model for the Intel RealSense 415 camera, in its
 aluminum peripherial evaluation case.
@@ -59,7 +46,6 @@
           <origin xyz="${d415_cam_mount_from_center_offset} ${-d415_cam_depth_py} 0" rpy="${M_PI/2} 0 ${M_PI/2}"/>
           <geometry>
-            <mesh filename="file://$(find realsense2_description)/meshes/d415.stl" />
+            <mesh filename="package://realsense2_description/meshes/d415.stl" />
           </geometry>
-          <material name="aluminum"/>
         </xacro:if>
         <xacro:unless value="${use_mesh}">
